File: midi/midi.kicad_sch (KiCad schematic)
At the start: 49 parts, among them J1 Conn_01x02, J2 SJ-43515TS-SMT-TR, J3 USB_C_Receptacle_USB2.0_16P, SW1 Reset, SW10 SW_Push, SW11 SW_Push, SW12 SW_Push, SW13 SW_Push, SW14 SW_Push, SW15 SW_Push, SW16 SW_Push, SW17 SW_Push, SW18 SW_Push, SW2 Boot, SW3 SW_Push, SW4 SW_Push, SW5 SW_Push, SW6 SW_Push, SW7 SW_Push, SW8 SW_Push, SW9 SW_Push, U1 ESP32-S2-SOLO, U2 SC189ZSKTRT, U3 MAX98357A, U4 MAX98357A, U5 CD74HC154M96

Commit message: add mounting holes, slight fixes, redo pours
Parts:
- added H1, H2, H3, H4: MountingHole, MountingHole:MountingHole_2.2mm_M2, symbol Mechanical:MountingHole
- U2: footprint SOT23-5-SC189_SEM -> SC189ZSKTRT:SOT23-5-SC189_SEM
Other:
- note added: "MOUNTING HOLES"
